Commit message: Added the stanford pupper URDF file, the mesh folder for the pupperV2 and a testing script to load the urdf in warp

File: urdf/standford_pupper.urdf (robot description, URDF)
Before this commit: robot stanford_pupper, 24 links, 23 joints
Links:
- link LF_HIP: geometry visual mesh filename=/teamspace/studios/this_studio/urdf/meshes/LF_HIP.STL
- link LF_THIGH: geometry visual mesh filename=/teamspace/studios/this_studio/urdf/meshes/LF_THIGH.STL
- link LF_THIGH_FOOT: geometry visual mesh filename=/teamspace/studios/this_studio/urdf/meshes/LF_THIGH_FOOT.STL
- link LH_HIP: geometry visual mesh filename=/teamspace/studios/this_studio/urdf/meshes/LH_HIP.STL
- link LH_THIGH: geometry visual mesh filename=/teamspace/studios/this_studio/urdf/meshes/LH_THIGH.STL
- link LH_THIGH_FOOT: geometry visual mesh filename=/teamspace/studios/this_studio/urdf/meshes/LH_THIGH_FOOT.STL
- link RF_HIP: geometry visual mesh filename=/teamspace/studios/this_studio/urdf/meshes/RF_HIP.STL
- link RF_THIGH: geometry visual mesh filename=/teamspace/studios/this_studio/urdf/meshes/RF_THIGH.STL
- link RF_THIGH_FOOT: geometry visual mesh filename=/teamspace/studios/this_studio/urdf/meshes/RF_THIGH_FOOT.STL
- link RH_HIP: geometry visual mesh filename=/teamspace/studios/this_studio/urdf/meshes/RH_HIP.STL
- link RH_THIGH: geometry visual mesh filename=/teamspace/studios/this_studio/urdf/meshes/RH_THIGH.STL
- link RH_THIGH_FOOT: geometry visual mesh filename=/teamspace/studios/this_studio/urdf/meshes/RH_THIGH_FOOT.STL
- link base_link: geometry collision mesh filename=/teamspace/studios/this_studio/urdf/meshes/base_link.STL; visual mesh filename=/teamspace/studios/this_studio/urdf/meshes/base_link.STL

Commit message: Remove large installer and re-commit

File: urdf/standford_pupper.urdf (robot description, URDF)
Before this commit: robot stanford_pupper, 24 links, 23 joints
Links:
- link LF_HIP: geometry visual mesh filename=meshes/LF_HIP.STL
- link LF_THIGH: geometry visual mesh filename=meshes/LF_THIGH.STL
- link LF_THIGH_FOOT: geometry visual mesh filename=meshes/LF_THIGH_FOOT.STL
- link LH_HIP: geometry visual mesh filename=meshes/LH_HIP.STL
- link LH_THIGH: geometry visual mesh filename=meshes/LH_THIGH.STL
- link LH_THIGH_FOOT: geometry visual mesh filename=meshes/LH_THIGH_FOOT.STL
- link RF_HIP: geometry visual mesh filename=meshes/RF_HIP.STL
- link RF_THIGH: geometry visual mesh filename=meshes/RF_THIGH.STL
- link RF_THIGH_FOOT: geometry visual mesh filename=meshes/RF_THIGH_FOOT.STL
- link RH_HIP: geometry visual mesh filename=meshes/RH_HIP.STL
- link RH_THIGH: geometry visual mesh filename=meshes/RH_THIGH.STL
- link RH_THIGH_FOOT: geometry visual mesh filename=meshes/RH_THIGH_FOOT.STL
- link base_link: geometry collision mesh filename=meshes/base_link.STL; visual mesh filename=meshes/base_link.STL

Commit message: Boxbox urdf test

File: urdf/standford_pupper.urdf (robot description, URDF)
Before this commit: robot stanford_pupper, 24 links, 23 joints
Links:
- removed link camera_depth_frame
- removed link camera_depth_optical_frame
- removed link camera_link
- removed link camera_rgb_frame
- removed link camera_rgb_optical_frame
- removed link hokuyo_frame
- removed link imu_link
Joints:
- removed joint camera_depth_joint
- removed joint camera_depth_optical_joint
- removed joint camera_joint
- removed joint camera_rgb_joint
- removed joint camera_rgb_optical_joint
- removed joint hokuyo_joint
- removed joint imu_joint
