Commit message: Update standford_pupper_clean.urdf

File: urdf/standford_pupper_clean.urdf (robot description, URDF)
Before this commit: robot stanford_pupper, 17 links, 16 joints
Links:
- link LF_THIGH: mass 0.00699575 -> 0.04
- link LF_THIGH_FOOT: mass 0.00294875 -> 0.03
- link LF_TOE: mass 0.002 -> 0.05
- link LH_THIGH: mass 0.00716530 -> 0.04
- link LH_THIGH_FOOT: mass 0.00294875 -> 0.03
- link LH_TOE: mass 0.002 -> 0.05
- link RF_THIGH: mass 0.00716529 -> 0.04
- link RF_THIGH_FOOT: mass 0.00294875 -> 0.03
- link RF_TOE: mass 0.002 -> 0.05
- link RH_THIGH: mass 0.00716529 -> 0.04
- link RH_THIGH_FOOT: mass 0.00294875 -> 0.03
- link RH_TOE: mass 0.002 -> 0.05
