Commit message: Created a new temp branch for the draft work, before pushing the clean setup in main.

File: artefacts/standford_pupper.urdf (robot description, URDF)
Before this commit: robot stanford_pupper, 24 links, 23 joints
Links:
- link LF_HIP: geometry collision box size=0.04 0.02 0.02; visual mesh filename=/teamspace/studios/this_studio/urdf/meshes/LF_HIP.STL
- link LF_THIGH: geometry collision capsule length=0.10 radius=0.015; visual mesh filename=/teamspace/studios/this_studio/urdf/meshes/LF_THIGH.STL
- link LF_THIGH_FOOT: geometry collision capsule length=0.12 radius=0.015; visual mesh filename=/teamspace/studios/this_studio/urdf/meshes/LF_THIGH_FOOT.STL
- link LF_TOE: geometry collision sphere radius=0.025; visual sphere radius=0.005
- link LH_HIP: geometry collision box size=0.04 0.02 0.02; visual mesh filename=/teamspace/studios/this_studio/urdf/meshes/LH_HIP.STL
- link LH_THIGH: geometry collision capsule length=0.10 radius=0.015; visual mesh filename=/teamspace/studios/this_studio/urdf/meshes/LH_THIGH.STL
- link LH_THIGH_FOOT: geometry collision capsule length=0.12 radius=0.015; visual mesh filename=/teamspace/studios/this_studio/urdf/meshes/LH_THIGH_FOOT.STL
- link LH_TOE: geometry collision sphere radius=0.025; visual sphere radius=0.005
- link RF_HIP: geometry collision box size=0.04 0.02 0.02; visual mesh filename=/teamspace/studios/this_studio/urdf/meshes/RF_HIP.STL
- link RF_THIGH: geometry collision capsule length=0.10 radius=0.015; visual mesh filename=/teamspace/studios/this_studio/urdf/meshes/RF_THIGH.STL
- link RF_THIGH_FOOT: geometry collision capsule length=0.12 radius=0.015; visual mesh filename=/teamspace/studios/this_studio/urdf/meshes/RF_THIGH_FOOT.STL
- link RF_TOE: geometry collision sphere radius=0.025; visual sphere radius=0.005
- link RH_HIP: geometry collision box size=0.04 0.02 0.02; visual mesh filename=/teamspace/studios/this_studio/urdf/meshes/RH_HIP.STL
- link RH_THIGH: geometry collision capsule length=0.10 radius=0.015; visual mesh filename=/teamspace/studios/this_studio/urdf/meshes/RH_THIGH.STL
- link RH_THIGH_FOOT: geometry collision capsule length=0.12 radius=0.015; visual mesh filename=/teamspace/studios/this_studio/urdf/meshes/RH_THIGH_FOOT.STL
- link RH_TOE: geometry collision sphere radius=0.025; visual sphere radius=0.005
- link base_link: geometry collision box size=0.3 0.15 0.1; visual mesh filename=/teamspace/studios/this_studio/urdf/meshes/base_link.STL
Joints:
- joint RH_HIP_JOINT: origin xyz=0.0705 -0.04 0.02425 rpy=0 0 0 -> xyz=-0.1299 -0.04 0.02425 rpy=0 0 0
- joint RH_THIGH_JOINT: origin xyz=-0.17265 -0.029523 0.0012724 rpy=-0.11522 0.436332 -0.1069 -> xyz=0.02775 -0.029523 0.0012724 rpy=-0.11522 0.436332 -0.1069
